File: simple/simple_record.brd (EAGLE design)
At the start: 8 parts, among them J1 SQUALL_HEADER, Q1 MOSFET-NCHANNELSMD, U2 MAX9939

Commit message: finalized title and some layout details
Parts:
- removed JP1: (no value), SparkFun-Connectors:1X02
- added JP2: (no value), SparkFun-Connectors:1X03
Connections:
- net GND: now also JP2.3; no longer JP1.2
- net INA-: now also JP2.1
- net PV+: now also JP2.2; no longer JP1.1
Routing:
- net INA-: track 6.46 -> 20.0 mm
- net PV+: track 17.8 -> 16.2 mm
- added copper zone on layer 16, net GND
Other:
- board text added: "GND"
- board text added: "IN+"
- board text added: "IN-"
Changed lines of the file:
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@@
 <board>
 <plain>
+<text x="9.2" y="1.1" size="1.016" layer="21">IN-</text>
+<text x="11.8" y="1.2" size="1.016" layer="21">IN+</text>
+<text x="14.6" y="1.3" size="1.016" layer="21">GND</text>
 </plain>
 <attributes>
@@
 </autorouter>
 <elements>
-<element name="U2" library="chips" package="UMAX10" value="MAX9939" x="10.16" y="8.89" rot="R270">
+<element name="U2" library="chips" package="UMAX10" value="MAX9939" x="10.16" y="8.89" smashed="yes" rot="R270">
 <attribute name="DIGIKEY" value="MAX9939AUB+-ND" x="-12.7" y="-24.13" size="1.778" layer="27" rot="R270" display="off"/>
-</element>
-<element name="JP1" library="SparkFun-Connectors" package="1X02" value="" x="11.43" y="3.81"/>
-<element name="Q1" library="fets" package="SOT23-3" value="MOSFET-NCHANNELSMD" x="7.62" y="12.7" rot="R90"/>
-<element name="R2" library="passives" package="0603-RES" value="100K" x="16.51" y="7.62" rot="R270"/>
-<element name="R3" library="passives" package="0603-RES" value="100K" x="16.51" y="11.43" rot="R270"/>
-<element name="C1" library="passives" package="0402_CAP" value="10uF" x="18.24" y="11.16" rot="R90"/>
-<element name="R1" library="passives" package="0603-RES" value="0.12" x="5.88" y="8.12" rot="R270"/>
-<element name="J1" library="squall" package="SQUALL_HEADER" value="SQUALL_HEADER" x="12.7" y="12.7">
+<attribute name="NAME" x="9.43" y="6.17" size="1.016" layer="21"/>
+</element>
+<element name="Q1" library="fets" package="SOT23-3" value="MOSFET-NCHANNELSMD" x="7.62" y="12.7" smashed="yes" rot="R90">
+<attribute name="NAME" x="7.7" y="15.742" size="1.016" layer="25" font="vector" ratio="12" rot="R180" align="bottom-center"/>
+</element>
+<element name="R2" library="passives" package="0603-RES" value="100K" x="16.51" y="7.62" smashed="yes" rot="R270">
+<attribute name="NAME" x="18.38" y="7.472" size="1.016" layer="25" font="vector" ratio="12" align="bottom-center"/>
+</element>
+<element name="R3" library="passives" package="0603-RES" value="100K" x="16.51" y="11.43" smashed="yes" rot="R270">
+<attribute name="NAME" x="16.47" y="12.772" size="1.016" layer="25" font="vector" ratio="12" align="bottom-center"/>
+</element>
+<element name="C1" library="passives" package="0402_CAP" value="10uF" x="18.24" y="11.16" smashed="yes" rot="R90">
+<attribute name="NAME" x="19.64" y="11.559" size="1.016" layer="25" font="vector" ratio="12" rot="R180" align="bottom-center"/>
+</element>
+<element name="R1" library="passives" package="0603-RES" value="0.12" x="5.88" y="8.12" smashed="yes" rot="R270">
+<attribute name="NAME" x="4.38" y="7.742" size="1.016" layer="25" font="vector" ratio="12" align="bottom-center"/>
+</element>
+<element name="J1" library="squall" package="SQUALL_HEADER" value="SQUALL_HEADER" x="12.7" y="12.7" smashed="yes">
 <attribute name="DIGIKEY" value="H11617CT-ND" x="12.7" y="12.7" size="1.778" layer="27" display="off"/>
+</element>
+<element name="JP2" library="SparkFun-Connectors" package="1X03" value="" x="10.3" y="3.8" smashed="yes">
+<attribute name="NAME" x="13.5538" y="5.2288" size="1.27" layer="25" ratio="10"/>
+<attribute name="VALUE" x="9.03" y="0.625" size="1.27" layer="27"/>
 </element>
 </elements>
 <signals>
 <signal name="GND">
-<contactref element="JP1" pad="2"/>
 <contactref element="Q1" pad="2"/>
 <contactref element="R3" pad="1"/>
@@
 <contactref element="J1" pad="A10"/>
 <polygon width="0.2032" layer="1" thermals="no">
-<vertex x="-1.4" y="22.7"/>
-<vertex x="-1.1" y="22.7"/>
-<vertex x="-1.1" y="-1.8"/>
-<vertex x="28.6" y="-1.8"/>
-<vertex x="28.6" y="24.6"/>
-<vertex x="-1.4" y="24.6"/>
+<vertex x="0" y="21.2"/>
+<vertex x="-0.1" y="-0.2"/>
+<vertex x="25.3" y="0"/>
+<vertex x="25.6" y="21"/>
 </polygon>
 <wire x1="1.855" y1="14.44" x2="4.495" y2="14.44" width="0.2032" layer="16"/>
@@
 <wire x1="6.2" y1="13.7" x2="8.57" y2="13.7" width="0.2032" layer="1"/>
 <wire x1="8.57" y1="13.7" x2="8.62" y2="13.65" width="0.2032" layer="1"/>
+<contactref element="JP2" pad="3"/>
+<polygon width="0.2032" layer="16" thermals="no">
+<vertex x="0" y="21.2"/>
+<vertex x="-0.1" y="-0.2"/>
+<vertex x="25.3" y="0"/>
+<vertex x="25.6" y="21"/>
+</polygon>
 </signal>
 <signal name="PV+">
-<contactref element="JP1" pad="1"/>
 <contactref element="R2" pad="2"/>
 <contactref element="U2" pad="5"/>
 <contactref element="R1" pad="2"/>
-<wire x1="11.43" y1="3.81" x2="8.29" y2="3.81" width="0.762" layer="1"/>
-<wire x1="8.29" y1="3.81" x2="5.8" y2="6.3" width="0.762" layer="1"/>
-<wire x1="5.8" y1="6.3" x2="5.8" y2="7.39" width="0.762" layer="1"/>
 <wire x1="5.8" y1="7.39" x2="5.88" y2="7.47" width="0.762" layer="1"/>
 <wire x1="5.88" y1="7.47" x2="6.87" y2="7.47" width="0.2032" layer="1"/>
@@
 <wire x1="7.3" y1="7.9" x2="7.98" y2="7.9" width="0.2032" layer="1"/>
 <wire x1="7.98" y1="7.9" x2="7.99" y2="7.89" width="0.2032" layer="1"/>
-<wire x1="11.43" y1="3.81" x2="11.43" y2="5.93" width="0.2032" layer="1"/>
-<wire x1="11.43" y1="5.93" x2="12.2" y2="6.7" width="0.2032" layer="1"/>
-<wire x1="12.2" y1="6.7" x2="16.24" y2="6.7" width="0.2032" layer="1"/>
 <wire x1="16.24" y1="6.7" x2="16.51" y2="6.97" width="0.2032" layer="1"/>
+<contactref element="JP2" pad="2"/>
+<wire x1="5.8" y1="7.39" x2="6.69" y2="6.5" width="0.508" layer="1"/>
+<wire x1="6.69" y1="6.5" x2="11.4" y2="6.5" width="0.508" layer="1"/>
+<wire x1="11.4" y1="6.5" x2="12.7" y2="5.2" width="0.508" layer="1"/>
+<wire x1="12.7" y1="5.2" x2="12.84" y2="5.06" width="0.508" layer="1"/>
+<wire x1="12.84" y1="5.06" x2="12.84" y2="3.8" width="0.508" layer="1"/>
+<wire x1="16.24" y1="6.7" x2="14.2" y2="6.7" width="0.2032" layer="1"/>
+<wire x1="14.2" y1="6.7" x2="12.7" y2="5.2" width="0.2032" layer="1"/>
 </signal>
 <signal name="INA-">
@@
 <contactref element="Q1" pad="3"/>
 <contactref element="R1" pad="1"/>
-<wire x1="5.88" y1="8.77" x2="5.88" y2="12.06" width="0.762" layer="1"/>
+<wire x1="5.88" y1="8.77" x2="5.88" y2="10" width="0.762" layer="1"/>
+<wire x1="5.88" y1="10" x2="5.88" y2="12.06" width="0.762" layer="1"/>
 <wire x1="5.88" y1="12.06" x2="6.52" y2="12.7" width="0.762" layer="1"/>
 <wire x1="5.88" y1="8.77" x2="6.93" y2="8.77" width="0.2032" layer="1"/>
@@
 <wire x1="7.3" y1="8.4" x2="7.98" y2="8.4" width="0.2032" layer="1"/>
 <wire x1="7.98" y1="8.4" x2="7.99" y2="8.39" width="0.2032" layer="1"/>
+<contactref element="JP2" pad="1"/>
+<wire x1="10.3" y1="3.8" x2="6.9" y2="3.8" width="0.508" layer="1"/>
+<wire x1="6.9" y1="3.8" x2="3.4" y2="7.3" width="0.508" layer="1"/>
+<wire x1="3.4" y1="7.3" x2="3.4" y2="9.8" width="0.508" layer="1"/>
+<wire x1="3.4" y1="9.8" x2="3.8" y2="10.2" width="0.508" layer="1"/>
+<wire x1="3.8" y1="10.2" x2="5.68" y2="10.2" width="0.508" layer="1"/>
+<wire x1="5.68" y1="10.2" x2="5.88" y2="10" width="0.508" layer="1"/>
 </signal>
 <signal name="CURRENT_SWITCH">
