File: simple/simple_record.sch (EAGLE design)
At the start: 8 parts, among them J1 SQUALL_HEADER, Q1 MOSFET-NCHANNELSMD, U2 MAX9939

Commit message: finalized title and some layout details
Parts:
- removed JP1: (no value), SparkFun-Connectors:M02PTH
- added JP2: (no value), SparkFun-Connectors:M03PTH
Connections:
- net GND: now also JP2.3; no longer JP1.2
- net INA-: now also JP2.1
- net PV+: now also JP2.2; no longer JP1.1
Other:
- note added: "Analog Circuitry to Sense Current and Voltage"
- note added: "Programmable Differential Gain Amplifier to Sense Current"
- note added: "Squall Header Connector"
- moved on the sheet: C1, J1, Q1, R1, R2, R3, U2
